File: myproject_uno/myproject_uno.kicad_pcb (KiCad board)
At the start: 2 copper layers, 68.6 x 53.3 mm, 8 parts, among them P1 Power, P2 Analog, P3 Digital, P4 Digital, P5 CONN_01X01, P6 CONN_01X01, P7 CONN_01X01, P8 CONN_01X01

Commit message: creation of first pcb kicad
Parts:
- added D1: LED, LED_SMD:LED_0201_0603Metric, F.Cu at (152.6, 110.2)
- added R1: R, Resistor_SMD:R_0201_0603Metric, F.Cu at (155.0, 110.2)
Routing:
- net /Vin: track 0.00 -> 14.2 mm
- net GND: track 0.00 -> 13.9 mm
- net Net-(D1-Pad2): track 0.00 -> 1.81 mm
Changed lines of the file:
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@@
-(kicad_pcb (version 4) (host pcbnew 4.0.2-4+6225~38~ubuntu14.04.1-stable)
+(kicad_pcb (version 20171130) (host pcbnew "(5.1.4)-1")
   (general
-    (links 4)
-    (no_connects 4)
-    (area 104.572999 71.392 182.146334 127.594)
     (thickness 1.6)
     (drawings 27)
-    (tracks 0)
+    (tracks 8)
     (zones 0)
-    (modules 8)
-    (nets 33)
+    (modules 10)
+    (nets 34)
   )
   (page A4)
@@
     (zone_45_only no)
     (trace_min 0.2)
-    (segment_width 0.15)
-    (edge_width 0.15)
     (via_size 0.6)
     (via_drill 0.4)
@@
     (uvia_min_size 0.2)
     (uvia_min_drill 0.1)
+    (edge_width 0.15)
+    (segment_width 0.15)
     (pcb_text_width 0.3)
     (pcb_text_size 1.5 1.5)
@@
     (pad_to_mask_clearance 0)
     (aux_axis_origin 110.998 126.365)
-    (grid_origin 110.998 126.365)
-    (visible_elements FFFFFF7F)
+    (visible_elements 7FFFFFFF)
     (pcbplotparams
       (layerselection 0x00030_80000001)
       (usegerberextensions false)
+      (usegerberattributes false)
+      (usegerberadvancedattributes false)
+      (creategerberjobfile false)
       (excludeedgelayer true)
       (linewidth 0.100000)
@@
       (hpglpennumber 1)
       (hpglpenspeed 20)
-      (hpglpendiameter 15)
-      (hpglpenoverlay 2)
+      (hpglpendiameter 15.000000)
       (psnegative false)
       (psa4output false)
@@
   (net 31 "/12(MISO)")
   (net 32 "/11(**/MOSI)")
+  (net 33 "Net-(D1-Pad2)")
   (net_class Default "This is the default net class."
     (clearance 0.2)
@@
     (add_net /Vin)
     (add_net GND)
+    (add_net "Net-(D1-Pad2)")
     (add_net "Net-(P1-Pad1)")
     (add_net "Net-(P5-Pad1)")
@@
       (net 5 /Vin))
     (model ${KIPRJMOD}/Socket_Arduino_Uno.3dshapes/Socket_header_Arduino_1x08.wrl
-      (at (xyz 0.35 0 0))
+      (offset (xyz 8.889999866485596 0 0))
       (scale (xyz 1 1 1))
       (rotate (xyz 0 0 180))
@@
       (net 12 "/A5(SCL)"))
     (model ${KIPRJMOD}/Socket_Arduino_Uno.3dshapes/Socket_header_Arduino_1x06.wrl
-      (at (xyz 0.25 0 0))
+      (offset (xyz 6.349999904632568 0 0))
       (scale (xyz 1 1 1))
       (rotate (xyz 0 0 180))
@@
       (net 14 /8))
     (model ${KIPRJMOD}/Socket_Arduino_Uno.3dshapes/Socket_header_Arduino_1x10.wrl
-      (at (xyz 0.45 0 0))
+      (offset (xyz 11.42999982833862 0 0))
       (scale (xyz 1 1 1))
       (rotate (xyz 0 0 180))
@@
       (net 22 "/0(Rx)"))
     (model ${KIPRJMOD}/Socket_Arduino_Uno.3dshapes/Socket_header_Arduino_1x08.wrl
-      (at (xyz 0.35 0 0))
+      (offset (xyz 8.889999866485596 0 0))
       (scale (xyz 1 1 1))
       (rotate (xyz 0 0 180))
@@
     (pad 1 thru_hole circle (at 0 0) (size 4.064 4.064) (drill 3.048) (layers *.Cu *.Mask F.SilkS)
       (net 26 "Net-(P8-Pad1)"))
+  )
+  (module LED_SMD:LED_0201_0603Metric (layer F.Cu)
+    (at 152.598001 110.230001)
+    (descr "LED SMD 0201 (0603 Metric), square (rectangular) end terminal, IPC_7351 nominal, (Body size source: https://www.vishay.com/docs/20052/crcw0201e3.pdf), generated with kicad-footprint-generator")
+    (tags LED)
+    (attr smd)
+    (fp_text reference D1 (at 0 -1.05) (layer F.SilkS)
+      (effects (font (size 1 1) (thickness 0.15)))
+    )
+    (fp_text value LED (at 0 1.05) (layer F.Fab)
+      (effects (font (size 1 1) (thickness 0.15)))
+    )
+    (fp_circle (center -0.86 0) (end -0.81 0) (layer F.SilkS) (width 0.1))
+    (fp_line (start -0.3 0.15) (end -0.3 -0.15) (layer F.Fab) (width 0.1))
+    (fp_line (start -0.3 -0.15) (end 0.3 -0.15) (layer F.Fab) (width 0.1))
+    (fp_line (start 0.3 -0.15) (end 0.3 0.15) (layer F.Fab) (width 0.1))
+    (fp_line (start 0.3 0.15) (end -0.3 0.15) (layer F.Fab) (width 0.1))
+    (fp_line (start -0.2 0.15) (end -0.2 -0.15) (layer F.Fab) (width 0.1))
+    (fp_line (start -0.1 0.15) (end -0.1 -0.15) (layer F.Fab) (width 0.1))
+    (fp_line (start -0.7 0.35) (end -0.7 -0.35) (layer F.CrtYd) (width 0.05))
+    (fp_line (start -0.7 -0.35) (end 0.7 -0.35) (layer F.CrtYd) (width 0.05))
+    (fp_line (start 0.7 -0.35) (end 0.7 0.35) (layer F.CrtYd) (width 0.05))
+    (fp_line (start 0.7 0.35) (end -0.7 0.35) (layer F.CrtYd) (width 0.05))
+    (fp_text user %R (at 0 -0.68) (layer F.Fab)
+      (effects (font (size 0.25 0.25) (thickness 0.04)))
+    )
+    (pad "" smd roundrect (at -0.345 0) (size 0.318 0.36) (layers F.Paste) (roundrect_rratio 0.25))
+    (pad "" smd roundrect (at 0.345 0) (size 0.318 0.36) (layers F.Paste) (roundrect_rratio 0.25))
+    (pad 1 smd roundrect (at -0.32 0) (size 0.46 0.4) (layers F.Cu F.Mask) (roundrect_rratio 0.25)
+      (net 4 GND))
+    (pad 2 smd roundrect (at 0.32 0) (size 0.46 0.4) (layers F.Cu F.Mask) (roundrect_rratio 0.25)
+      (net 33 "Net-(D1-Pad2)"))
+    (model ${KISYS3DMOD}/LED_SMD.3dshapes/LED_0201_0603Metric.wrl
+      (at (xyz 0 0 0))
+      (scale (xyz 1 1 1))
+      (rotate (xyz 0 0 0))
+    )
+  )
+  (module Resistor_SMD:R_0201_0603Metric (layer F.Cu)
+    (at 155.043001 110.230001 180)
+    (descr "Resistor SMD 0201 (0603 Metric), square (rectangular) end terminal, IPC_7351 nominal, (Body size source: https://www.vishay.com/docs/20052/crcw0201e3.pdf), generated with kicad-footprint-generator")
+    (tags resistor)
+    (attr smd)
+    (fp_text reference R1 (at 0 -1.05) (layer F.SilkS)
+      (effects (font (size 1 1) (thickness 0.15)))
+    )
+    (fp_text value R (at 0 1.05) (layer F.Fab)
+      (effects (font (size 1 1) (thickness 0.15)))
+    )
+    (fp_line (start -0.3 0.15) (end -0.3 -0.15) (layer F.Fab) (width 0.1))
+    (fp_line (start -0.3 -0.15) (end 0.3 -0.15) (layer F.Fab) (width 0.1))
+    (fp_line (start 0.3 -0.15) (end 0.3 0.15) (layer F.Fab) (width 0.1))
+    (fp_line (start 0.3 0.15) (end -0.3 0.15) (layer F.Fab) (width 0.1))
+    (fp_line (start -0.7 0.35) (end -0.7 -0.35) (layer F.CrtYd) (width 0.05))
+    (fp_line (start -0.7 -0.35) (end 0.7 -0.35) (layer F.CrtYd) (width 0.05))
+    (fp_line (start 0.7 -0.35) (end 0.7 0.35) (layer F.CrtYd) (width 0.05))
+    (fp_line (start 0.7 0.35) (end -0.7 0.35) (layer F.CrtYd) (width 0.05))
+    (fp_text user %R (at 0 -0.68) (layer F.Fab)
+      (effects (font (size 0.25 0.25) (thickness 0.04)))
+    )
+    (pad "" smd roundrect (at -0.345 0 180) (size 0.318 0.36) (layers F.Paste) (roundrect_rratio 0.25))
+    (pad "" smd roundrect (at 0.345 0 180) (size 0.318 0.36) (layers F.Paste) (roundrect_rratio 0.25))
+    (pad 1 smd roundrect (at -0.32 0 180) (size 0.46 0.4) (layers F.Cu F.Mask) (roundrect_rratio 0.25)
+      (net 5 /Vin))
+    (pad 2 smd roundrect (at 0.32 0 180) (size 0.46 0.4) (layers F.Cu F.Mask) (roundrect_rratio 0.25)
+      (net 33 "Net-(D1-Pad2)"))
+    (model ${KISYS3DMOD}/Resistor_SMD.3dshapes/R_0201_0603Metric.wrl
+      (at (xyz 0 0 0))
+      (scale (xyz 1 1 1))
+      (rotate (xyz 0 0 0))
+    )
   )
   (gr_text 1 (at 138.938 121.285 90) (layer F.SilkS)
@@
   (gr_line (start 120.523 82.55) (end 120.523 93.98) (angle 90) (layer Dwgs.User) (width 0.15))
   (gr_line (start 104.648 82.55) (end 120.523 82.55) (angle 90) (layer Dwgs.User) (width 0.15))
+  (segment (start 152.278001 123.184999) (end 151.638 123.825) (width 0.25) (layer F.Cu) (net 4))
+  (segment (start 152.278001 110.230001) (end 152.278001 123.184999) (width 0.25) (layer F.Cu) (net 4))
+  (segment (start 156.718 123.6726) (end 156.718 123.825) (width 0.25) (layer F.Cu) (net 5))
+  (segment (start 155.6044 122.559) (end 156.718 123.6726) (width 0.25) (layer F.Cu) (net 5))
+  (segment (start 155.452 122.559) (end 155.6044 122.559) (width 0.25) (layer F.Cu) (net 5))
+  (segment (start 155.363001 122.470001) (end 155.452 122.559) (width 0.25) (layer F.Cu) (net 5))
+  (segment (start 155.363001 110.230001) (end 155.363001 122.470001) (width 0.25) (layer F.Cu) (net 5))
+  (segment (start 152.918001 110.230001) (end 154.723001 110.230001) (width 0.25) (layer F.Cu) (net 33))
 )
